Commit message: Added a yellow triangle to workspace.

File: workspace/ros2_ws/src/panda_env/panda_env/gym_example/gym_example/envs/objects/triangle_yellow.urdf (robot description, URDF)
Before this commit: robot triangle.urdf, 1 links, 0 joints
Links:
- link baseLink: geometry collision mesh filename=triangle.obj scale=0.7 1 1; visual mesh filename=triangle.obj scale=0.7 1 1
