Commit message: Fixed rotations

File: workspace/ros2_ws/src/panda_env/panda_env/gym_example/gym_example/envs/objects/cube_blue.urdf (robot description, URDF)
Before this commit: robot cube_blue, 1 links, 0 joints
Links:
- link baseLink: mass 1.0 -> 0.1; geometry collision box size=0.05 0.05 0.05; visual mesh filename=cube.obj scale=0.05 0.05 0.05

File: workspace/ros2_ws/src/panda_env/panda_env/gym_example/gym_example/envs/objects/cube_green.urdf (robot description, URDF)
Before this commit: robot cube_green, 1 links, 0 joints
Links:
- link baseLink: mass 1.0 -> 0.1; geometry collision box size=0.05 0.05 0.05; visual mesh filename=cube.obj scale=0.05 0.05 0.05

File: workspace/ros2_ws/src/panda_env/panda_env/gym_example/gym_example/envs/objects/cube_red.urdf (robot description, URDF)
Before this commit: robot cube_red, 1 links, 0 joints
Links:
- link baseLink: mass 1.0 -> 0.1; geometry collision box size=0.05 0.05 0.05; visual mesh filename=cube.obj scale=0.05 0.05 0.05
