Commit message: Added cylinders and bricks. Restructured the objects.

File: workspace/ros2_ws/src/panda_env/panda_env/gym_example/gym_example/envs/base_objects/brick.urdf (robot description, URDF)
Before this commit: robot cube_green, 1 links, 0 joints
Links:
- link baseLink: mass 1.0 -> .1; geometry collision box size=.05 .15 .05; visual mesh filename=brick.obj scale=.05 .15 .05

File: workspace/ros2_ws/src/panda_env/panda_env/gym_example/gym_example/envs/workspace_objects/brick_cyan.urdf (robot description, URDF)
Before this commit: robot cube, 1 links, 0 joints
Links:
- link baseLink: mass 1.0 -> .1; geometry collision box size=.05 .15 .05; visual mesh filename=../base_objects/brick.obj scale=.05 .15 .05

File: workspace/ros2_ws/src/panda_env/panda_env/gym_example/gym_example/envs/workspace_objects/cube_blue.urdf (robot description, URDF)
Before this commit: robot cube_red, 1 links, 0 joints
Links:
- link baseLink: geometry collision box size=1 1 1; visual mesh filename=../base_objects/cube.obj scale=0.05 0.05 0.05

File: workspace/ros2_ws/src/panda_env/panda_env/gym_example/gym_example/envs/workspace_objects/cube_green.urdf (robot description, URDF)
Before this commit: robot cube_blue, 1 links, 0 joints
Links:
- link baseLink: geometry collision box size=1 1 1; visual mesh filename=../base_objects/cube.obj scale=0.05 0.05 0.05

File: workspace/ros2_ws/src/panda_env/panda_env/gym_example/gym_example/envs/workspace_objects/triangle_yellow.urdf (robot description, URDF)
Before this commit: robot triangle.urdf, 1 links, 0 joints
Links:
- link baseLink: geometry collision mesh filename=../base_objects/triangle.obj scale=0.7 1 1; visual mesh filename=../base_objects/triangle.obj scale=0.7 1 1
